File: hardware/Badge-Pwnterrey-2026.kicad_sch (KiCad schematic)
At the start: 23 parts, among them P1 USB_C_Plug_USB2.0, SW1 RESET, SW2 GPIO, U1 ESP32-C5-WROOM-1-N4, U2 AP2112K-3.3, U3 NT3H2111W0FHK

Commit message: feat(Hw):Init_Floorplan
Parts:
- added SW3: On, Footprints:MSK12C02, symbol Switch:SW_DPDT_x2
Connections:
- net EPAD: now also SW3.4 (C)
- net VBUS: now also SW3.1 (A); no longer C9.1, U2.1 (VIN), U2.3 (EN)
- new net: C9.1, SW3.2 (B), U2.1 (VIN), U2.3 (EN)
- no-connect marks 18 -> 19
Changed lines of the file:
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@@
 	)
 	(junction
-		(at 43.18 175.006)
+		(at 124.46 153.67)
 		(diameter 0)
 		(color 0 0 0 0)
 	)
 	(junction
-		(at 233.68 77.47)
+		(at 43.18 175.006)
 		(diameter 0)
 		(color 0 0 0 0)
 	)
 	(junction
-		(at 233.68 42.164)
+		(at 233.68 77.47)
 		(diameter 0)
 		(color 0 0 0 0)
 	)
 	(junction
-		(at 213.36 45.974)
+		(at 233.68 42.164)
 		(diameter 0)
 		(color 0 0 0 0)
 	)
 	(junction
-		(at 124.46 153.67)
+		(at 213.36 45.974)
 		(diameter 0)
 		(color 0 0 0 0)
@@
 	)
 	(no_connect
+		(at 109.22 151.13)
+	)
+	(no_connect
 		(at 38.1 73.66)
 	)
@@
 	(wire
 		(pts
+			(xy 119.38 153.67) (xy 124.46 153.67)
+		)
+		(stroke
+			(width 0)
+			(type default)
+		)
+	)
+	(wire
+		(pts
 			(xy 220.98 45.974) (xy 213.36 45.974)
 		)
@@
 	(wire
 		(pts
-			(xy 120.65 153.67) (xy 124.46 153.67)
+			(xy 100.33 156.21) (xy 109.22 156.21)
 		)
 		(stroke
@@
 	(wire
 		(pts
+			(xy 107.95 147.32) (xy 109.22 147.32)
+		)
+		(stroke
+			(width 0)
+			(type default)
+		)
+	)
+	(wire
+		(pts
 			(xy 35.56 60.96) (xy 38.1 60.96)
 		)
@@
 	(wire
 		(pts
-			(xy 120.65 151.13) (xy 120.65 153.67)
+			(xy 100.33 153.67) (xy 100.33 156.21)
 		)
 		(stroke
@@
 		)
 	)
+	(label "GND"
+		(at 107.95 147.32 180)
+		(effects
+			(font
+				(size 1.27 1.27)
+			)
+			(justify right bottom)
+		)
+	)
 	(label "SCL"
 		(at 259.08 128.27 270)
@@
 	(symbol
 		(lib_id "power:VBUS")
-		(at 120.65 151.13 0)
+		(at 100.33 153.67 0)
 		(unit 1)
 		(exclude_from_sim no)
@@
 		(dnp no)
 		(property "Reference" "#PWR09"
-			(at 120.65 154.94 0)
+			(at 100.33 157.48 0)
 			(effects
 				(font
@@
 		)
 		(property "Value" "VBUS"
-			(at 121.031 146.7358 0)
+			(at 100.711 149.2758 0)
 			(effects
 				(font
@@
 		)
 		(property "Footprint" ""
-			(at 120.65 151.13 0)
+			(at 100.33 153.67 0)
 			(effects
 				(font
@@
 		)
 		(property "Datasheet" ""
-			(at 120.65 151.13 0)
+			(at 100.33 153.67 0)
 			(effects
 				(font
@@
 		)
 		(property "Description" ""
-			(at 120.65 151.13 0)
+			(at 100.33 153.67 0)
 			(effects
 				(font
@@
 					(unit 1)
 				)
+			)
+		)
+	)
+	(symbol
+		(lib_id "Switch:SW_DPDT_x2")
+		(at 114.3 153.67 180)
+		(unit 1)
+		(exclude_from_sim no)
+		(in_bom yes)
+		(on_board yes)
+		(dnp no)
+		(property "Reference" "SW3"
+			(at 116.078 150.241 0)
+			(effects
+				(font
+					(size 1.27 1.27)
+				)
+			)
+		)
+		(property "Value" "On"
+			(at 114.3 158.5976 0)
+			(effects
+				(font
+					(size 1.27 1.27)
+				)
+			)
+		)
+		(property "Footprint" "Footprints:MSK12C02"
+			(at 114.3 153.67 0)
+			(effects
+				(font
+					(size 1.27 1.27)
+				)
+				(hide yes)
+			)
+		)
+		(property "Datasheet" "~"
+			(at 114.3 153.67 0)
+			(effects
+				(font
+					(size 1.27 1.27)
+				)
+				(hide yes)
+			)
+		)
+		(property "Description" ""
+			(at 114.3 153.67 0)
+			(effects
+				(font
+					(size 1.27 1.27)
+				)
+				(hide yes)
+			)
+		)
+		(property "LCSC#" "C431540"
+			(at 114.3 153.67 0)
+			(effects
+				(font
+					(size 1.27 1.27)
+				)
+				(hide yes)
+			)
+		)
+		(property "manf#" ""
+			(at 114.3 153.67 0)
+			(effects
+				(font
+					(size 1.27 1.27)
+				)
+				(hide yes)
+			)
+		)
+		(pin "1"
+		)
+		(pin "2"
+		)
+		(pin "3"
+		)
+		(pin "4"
+		)
+		(pin "5"
+		)
+		(pin "6"
+		)
+		(pin "4"
+		)
+		(instances
+			(project "Badge-Pwnterrey-2026"
+				(path "/e3b2b1fe-149a-4e04-8ccb-2dcccbdaccab"
+					(reference "SW3")
+					(unit 1)
+				)
