File: hardware/Badge-Pwnterrey-2026.kicad_sch (KiCad schematic)
At the start: 42 parts, among them J1 Conn_01x08_Socket, J2 Conn_01x08_Socket, J3 Conn_01x10_Socket, J5 Conn_01x10_Socket, P1 USB_C_Plug_USB2.0, Q1 DMP2004TK-7, Q2 DMP2004TK-7, SW1 RESET, SW2 GPIO, SW3 On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

Commit message: feat(Hw):Update_Labels
Other:
- company: (none) -> Electronic Cats
- title: (none) -> Badge-Pwnterrey-2026
Changed lines of the file:
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@@
 	(generator_version "9.0")
 	(paper "A4")
+	(title_block
+		(title "Badge-Pwnterrey-2026")
+		(date "2026-03-23")
+		(rev "v1.0")
+		(company "Electronic Cats")
+		(comment 1 "Lizeth Gallegos Martínez")
+	)
 	(text "PB2"
 		(exclude_from_sim no)

Commit message: feat(Hw):Update_Schematic_And_Route
Connections:
- net RX: now also U5.3 (RXD); no longer U5.2 (TXD)
- net TX: now also U5.2 (TXD); no longer U5.3 (RXD)
Changed lines of the file:
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@@
 	(wire
 		(pts
-			(xy 119.634 182.88) (xy 118.11 182.88)
-		)
-		(stroke
-			(width 0)
-			(type default)
-		)
-	)
-	(wire
-		(pts
 			(xy 51.308 109.22) (xy 51.308 111.76)
 		)
@@
 	(wire
 		(pts
-			(xy 119.634 185.42) (xy 118.11 185.42)
-		)
-		(stroke
-			(width 0)
-			(type default)
-		)
-	)
-	(wire
-		(pts
 			(xy 195.58 120.65) (xy 195.58 128.27)
 		)
@@
 	(wire
 		(pts
+			(xy 118.11 185.42) (xy 119.38 185.42)
+		)
+		(stroke
+			(width 0)
+			(type default)
+		)
+	)
+	(wire
+		(pts
 			(xy 81.534 184.658) (xy 81.534 184.15)
 		)
@@
 	(wire
 		(pts
+			(xy 118.11 182.88) (xy 119.38 182.88)
+		)
+		(stroke
+			(width 0)
+			(type default)
+		)
+	)
+	(wire
+		(pts
 			(xy 87.376 184.658) (xy 87.376 172.72)
 		)
@@
 	)
 	(label "TX"
-		(at 119.634 182.88 0)
+		(at 119.38 185.42 0)
 		(effects
 			(font
@@
 	)
 	(label "RX"
-		(at 119.634 185.42 0)
+		(at 119.38 182.88 0)
 		(effects
 			(font
@@
 					(size 1.27 1.27)
 				)
+				(hide yes)
 			)
 		)
 		(property "Footprint" "Footprints:AT2659S-LSA"
-			(at 58.674 174.244 0)
+			(at 58.928 182.118 0)
 			(effects
 				(font
@@
 		)
 		(property "Datasheet" "https://datasheet.lcsc.com/lcsc/2109191430_ZHONGKEWEI-AT2659S_C883443.pdf"
-			(at 58.674 174.244 0)
+			(at 58.42 181.864 0)
 			(effects
 				(font
@@
 		)
 		(property "LCSC#" "C883443"
-			(at 65.024 174.244 0)
+			(at 65.278 182.118 0)
 			(effects
 				(font

Commit message: feat(Hw):Update_Schematic_And_Route
Connections:
- net RX: no longer U5.3 (RXD)
- net TX: no longer U5.2 (TXD)
- net GPS_TX: now reaches U1.23 (IO24)
- net GPS_TX: now also U5.2 (TXD)
- net GPS_RX: now reaches U1.26 (IO25)
- net GPS_RX: now also U5.3 (RXD)
- no-connect marks 14 -> 12
Other:
- moved on the sheet: C14
Changed lines of the file:
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@@
 	)
 	(junction
-		(at 125.222 187.96)
+		(at 129.54 187.96)
 		(diameter 0)
 		(color 0 0 0 0)
@@
 	)
 	(junction
-		(at 125.222 175.26)
+		(at 129.54 175.26)
 		(diameter 0)
 		(color 0 0 0 0)
@@
 	)
 	(junction
-		(at 125.222 170.18)
+		(at 129.54 170.18)
 		(diameter 0)
 		(color 0 0 0 0)
@@
 	)
 	(no_connect
-		(at 77.47 57.15)
-	)
-	(no_connect
-		(at 77.47 59.69)
-	)
-	(no_connect
 		(at 36.83 46.99)
 	)
@@
 	(wire
 		(pts
-			(xy 118.11 175.26) (xy 125.222 175.26)
+			(xy 118.11 175.26) (xy 129.54 175.26)
 		)
 		(stroke
@@
 	(wire
 		(pts
-			(xy 125.222 170.18) (xy 125.222 175.26)
+			(xy 129.54 170.18) (xy 129.54 175.26)
 		)
 		(stroke
@@
 	(wire
 		(pts
+			(xy 85.09 57.15) (xy 77.47 57.15)
+		)
+		(stroke
+			(width 0)
+			(type default)
+		)
+	)
+	(wire
+		(pts
 			(xy 227.33 48.26) (xy 227.33 46.99)
 		)
@@
 	(wire
 		(pts
-			(xy 125.222 184.15) (xy 125.222 187.96)
+			(xy 129.54 184.15) (xy 129.54 187.96)
 		)
 		(stroke
@@
 	(wire
 		(pts
-			(xy 125.222 175.26) (xy 125.222 179.07)
+			(xy 129.54 175.26) (xy 129.54 179.07)
 		)
 		(stroke
@@
 	(wire
 		(pts
-			(xy 118.11 187.96) (xy 125.222 187.96)
+			(xy 118.11 187.96) (xy 129.54 187.96)
 		)
 		(stroke
@@
 	(wire
 		(pts
-			(xy 125.222 187.96) (xy 125.222 189.738)
+			(xy 129.54 187.96) (xy 129.54 189.738)
 		)
 		(stroke
@@
 	(wire
 		(pts
-			(xy 125.222 169.672) (xy 125.222 170.18)
+			(xy 129.54 169.672) (xy 129.54 170.18)
 		)
 		(stroke
@@
 	(wire
 		(pts
-			(xy 118.11 170.18) (xy 125.222 170.18)
+			(xy 118.11 170.18) (xy 129.54 170.18)
 		)
 		(stroke
@@
 	(wire
 		(pts
+			(xy 85.09 59.69) (xy 77.47 59.69)
+		)
+		(stroke
+			(width 0)
+			(type default)
+		)
+	)
+	(wire
+		(pts
 			(xy 229.87 62.23) (xy 231.14 62.23)
 		)
@@
 		)
 	)
+	(label "GPS_RX"
+		(at 85.09 59.69 180)
+		(effects
+			(font
+				(size 1.27 1.27)
+			)
+			(justify right bottom)
+		)
+	)
 	(label "RST"
 		(at 124.46 37.084 0)
@@
 		)
 	)
-	(label "TX"
+	(label "GPS_TX"
 		(at 119.38 185.42 0)
 		(effects
@@
 		)
 	)
+	(label "GPS_TX"
+		(at 85.09 57.15 180)
+		(effects
+			(font
+				(size 1.27 1.27)
+			)
+			(justify right bottom)
+		)
+	)
 	(label "D-"
 		(at 43.18 116.84 0)
@@
 		)
 	)
-	(label "RX"
+	(label "GPS_RX"
 		(at 119.38 182.88 0)
 		(effects
@@
 	(symbol
 		(lib_id "power:+3V3")
-		(at 125.222 169.672 0)
+		(at 129.54 169.672 0)
 		(unit 1)
 		(exclude_from_sim no)
@@
 		(dnp no)
 		(property "Reference" "#PWR034"
-			(at 125.222 173.482 0)
+			(at 129.54 173.482 0)
 			(effects
 				(font
@@
 		)
 		(property "Value" "+3V3"
-			(at 125.603 165.2778 0)
+			(at 129.921 165.2778 0)
 			(effects
 				(font
@@
 		)
 		(property "Footprint" ""
-			(at 125.222 169.672 0)
+			(at 129.54 169.672 0)
 			(effects
 				(font
@@
 		)
 		(property "Datasheet" ""
-			(at 125.222 169.672 0)
+			(at 129.54 169.672 0)
 			(effects
 				(font
@@
 		)
 		(property "Description" ""
-			(at 125.222 169.672 0)
+			(at 129.54 169.672 0)
 			(effects
 				(font
@@
 	(symbol
 		(lib_id "Device:C_Small")
-		(at 125.222 181.61 180)
+		(at 129.54 181.61 180)
 		(unit 1)
 		(exclude_from_sim no)
@@
 		(dnp no)
 		(property "Reference" "C14"
-			(at 126.238 177.038 90)
+			(at 130.556 177.038 90)
 			(effects
 				(font
@@
 		)
 		(property "Value" "10uF"
-			(at 128.016 179.578 90)
+			(at 132.334 179.578 90)
 			(effects
 				(font
@@
 		)
 		(property "Footprint" "Capacitor_SMD:C_0603_1608Metric"
-			(at 125.222 181.61 0)
+			(at 129.54 181.61 0)
 			(effects
 				(font
@@
 		)
 		(property "Datasheet" "https://datasheet.lcsc.com/lcsc/1912111437_CCTC-TCC0603COG100J500CT_C376764.pdf"
-			(at 125.222 181.61 0)
+			(at 129.54 181.61 0)
 			(effects
 				(font
@@
 		)
 		(property "Description" ""
-			(at 125.222 181.61 0)
+			(at 129.54 181.61 0)
 			(effects
 				(font
@@
 		)
 		(property "manf#" ""
-			(at 125.222 181.61 0)
+			(at 129.54 181.61 0)
 			(effects
 				(font
@@
 		)
 		(property "provedor" "LCSC"
-			(at 125.222 181.61 0)
+			(at 129.54 181.61 0)
 			(effects
 				(font
@@
 		)
 		(property "LCSC#" "C85713"
-			(at 125.222 181.61 0)
+			(at 129.54 181.61 0)
 			(effects
 				(font
@@
 	(symbol
 		(lib_id "power:GND")
-		(at 125.222 189.738 0)
+		(at 129.54 189.738 0)
 		(unit 1)
 		(exclude_from_sim no)
@@
 		(dnp no)
 		(property "Reference" "#PWR036"
-			(at 125.222 196.088 0)
+			(at 129.54 196.088 0)
 			(effects
 				(font
@@
 		)
 		(property "Value" "GND"
-			(at 125.349 194.1322 0)
+			(at 129.667 194.1322 0)
 			(effects
 				(font
@@
 		)
 		(property "Footprint" ""
-			(at 125.222 189.738 0)
+			(at 129.54 189.738 0)
 			(effects
 				(font
@@
 		)
 		(property "Datasheet" ""
-			(at 125.222 189.738 0)
+			(at 129.54 189.738 0)
 			(effects
 				(font
@@
 		)
 		(property "Description" ""
-			(at 125.222 189.738 0)
+			(at 129.54 189.738 0)
 			(effects
 				(font

Commit message: feat(Hw):Update_Schematic_And_Route
Parts:
- added D1: MBR120, Diode_SMD:D_SOD-123F, symbol Diode:MBR340
- added Q3: DMG3415U-7, Package_TO_SOT_SMD:SOT-23, symbol Device:Q_PMOS_GSD
- added R5: 100K, Resistor_SMD:R_0603_1608Metric, symbol Device:R_Small
Connections:
- net +3V3: now also SW3.2 (B); no longer C2.1, C25.1, J3.10 (Pin_1), J5.10 (Pin_1), U2.5 (VOUT)
- net EPAD: now also R5.2
- net VBUS: now also C9.1, U2.1 (VIN), U2.3 (EN); no longer SW3.1 (A)
- new net: C25.1, D1.2 (A), Q3.1 (G), R5.1, U2.5 (VOUT)
- new net: D1.1 (K), Q3.2 (S), SW3.1 (A)
- new net +3.3V: C2.1, J3.10 (Pin_1), J5.10 (Pin_1), Q3.3 (D)
Other:
- moved on the sheet: C2, C25, C9, SW3A, U2

Commit message: feat(hw):Added_TPS2116DRL
Parts:
- removed C25, C9: 10uF, Capacitor_SMD:C_0603_1608Metric, symbol Device:C_Small
- removed D1: MBR120, Diode_SMD:D_SOD-123F, symbol Diode:MBR340
- removed Q3: DMG3415U-7, Package_TO_SOT_SMD:SOT-23, symbol Device:Q_PMOS_GSD
- removed R5: 100K, Resistor_SMD:R_0603_1608Metric, symbol Device:R_Small
- added C7, C8: 10uF, Capacitor_SMD:C_0603_1608Metric, symbol Device:C_Small
- added R10: 4.7k, Resistor_SMD:R_0603_1608Metric, symbol Device:R
- added R12, R5: 10k, Resistor_SMD:R_0603_1608Metric, symbol Device:R
- added U7: TPS2116DRL, Package_TO_SOT_SMD:SOT-583-8, symbol Power_Management:TPS2116DRL
Connections:
- net +3.3V: now also U7.6 (VIN2)
- net EPAD: now also C7.2, C8.2, R12.2, U7.1 (GND)
- net VBUS: now also C7.1
- net Vref: now reaches U2.5 (VOUT)
- net Vref: now also C8.1, R10.1, U7.3 (VIN1), U7.5 (MODE)
- net at SW3.1 (A): now also R5.1, U7.2 (VOUT), U7.7 (VOUT)
- new net: R5.2, U7.8 (ST)
- new net PR1: R10.2, R12.1, U7.4 (PR1)
Other:
- moved on the sheet: SW3A

Commit message: feat(Hw):Update_Schematic_And_Route
Parts:
- added C9: 100nF, Capacitor_SMD:C_0603_1608Metric, symbol Device:C_Small
- J1, J2: LCSC# C492407 -> C49326132
- J3, J5: LCSC# C57369 -> C49326134
Connections:
- net EPAD: now also C9.1
- net at R5.1, SW3.1 (A), U7.2 (VOUT)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: now also C9.2
Other:
- moved on the sheet: C10, C11, C7, C8, F1, L1, P1, R10, R12, R15, R16, R17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

Commit message: feat(Hw):Update_BOM
Parts:
- J1, J3: now not fitted
Changed lines of the file:
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@@
 		(in_bom yes)
 		(on_board yes)
-		(dnp no)
+		(dnp yes)
 		(property "Reference" "J1"
 			(at 235.585 26.289 0)
@@
 		(in_bom yes)
 		(on_board yes)
-		(dnp no)
+		(dnp yes)
 		(property "Reference" "J3"
 			(at 235.077 57.658 0)

Commit message: feat(Hw):GPS_Pins_Added
Parts:
- added J4: GPS, Connector_PinHeader_2.54mm:PinHeader_1x04_P2.54mm_Vertical, symbol Connector_Generic:Conn_01x04
Connections:
- net +3V3: now also J4.1 (Pin_1)
- net EPAD: now also J4.4 (Pin_4)
- net GPS_RX: now also J4.2 (Pin_2)
- net GPS_TX: now also J4.3 (Pin_3)
Other:
- moved on the sheet: AE1, C14, C15, C6, L2, U4, U5
