File: hardware/Badge-Pwnterrey-2026.kicad_pcb (KiCad board)
At the start: 2 copper layers, 75.5 x 60.2 mm, 60 parts, among them J1 Conn_01x08_Socket, J2 Conn_01x08_Socket, J3 Conn_01x10_Socket, J5 Conn_01x10_Socket, P1 USB_C_Plug_USB2.0, Q1 DMP2004TK-7, Q2 DMP2004TK-7, SW1 RESET, SW2 GPIO, SW3 On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

Commit message: feat(Hw):Update_Schematic_And_Route
Parts:
- moved R17 0.50 mm to (146.6, 64.0)
- moved C10 0.50 mm to (144.2, 68.4)
- moved R16 0.50 mm to (144.7, 61.6)
- moved L1 0.50 mm to (126.6, 64.5)
- moved C11 0.50 mm to (142.0, 64.5)
- moved R15 0.50 mm to (145.6, 68.4)
- moved U3 0.50 mm to (144.2, 64.8)
Connections:
- U5 pad 2: /RX -> /TX
- U5 pad 3: /TX -> /RX
Routing:
- net GND: track 6.54 -> 18.1 mm, vias 81 -> 80
- net /RX: track 74.3 -> 76.3 mm
- net /TX: track 82.6 -> 81.6 mm

Commit message: feat(Hw):Update_Schematic_And_Route
Connections:
- U1 pad 23: unconnected-(U1-IO24-Pad23) -> /GPS_TX
- U1 pad 26: unconnected-(U1-IO25-Pad26) -> /GPS_RX
- U5 pad 2: /TX -> /GPS_TX
- U5 pad 3: /RX -> /GPS_RX
Routing:
- net /GPS_RX: track 0.00 -> 45.7 mm, vias 0 -> 2
- net /GPS_TX: track 0.00 -> 40.0 mm, vias 0 -> 2
- net /TX: track 81.6 -> 59.1 mm, vias 2 -> 1
- net /RX: track 76.3 -> 61.8 mm, vias 3 -> 1
- net /SWDIO: vias 1 -> 2
- net GND: vias 80 -> 85

Commit message: feat(Hw):Update_Schematic_And_Route
Parts:
- added D1: MBR120, Diode_SMD:D_SOD-123F, B.Cu at (122.6, 90.7)
- added Q3: DMG3415U-7, Package_TO_SOT_SMD:SOT-23, B.Cu at (125.9, 90.7)
- added R5: 100K, Resistor_SMD:R_0603_1608Metric, B.Cu at (123.4, 93.8)
- moved C9 9.95 mm to (128.8, 96.8), turned to -90 degrees
- moved C25 7.76 mm to (122.4, 96.7), turned to -90 degrees
- moved U2 6.20 mm to (125.5, 96.7), turned to 180 degrees
Connections:
- C2 pad 1: +3V3 -> +3.3V
- C25 pad 1: +3V3 -> Net-(D1-A)
- C9 pad 1: Net-(SW3A-B) -> VBUS
- J3 pad 10: +3V3 -> +3.3V
- J5 pad 10: +3V3 -> +3.3V
- SW3 pad 1: VBUS -> Net-(D1-K)
- SW3 pad 2: Net-(SW3A-B) -> +3V3
- U2 pad 1: Net-(SW3A-B) -> VBUS
- U2 pad 3: Net-(SW3A-B) -> VBUS
- U2 pad 5: +3V3 -> Net-(D1-A)
Routing:
- net +3.3V: track 0.00 -> 40.7 mm
- net +3V3: track 206.0 -> 188.9 mm
- net Net-(D1-K): track 0.00 -> 12.0 mm
- net Net-(SW3A-B): track 10.5 -> 0.00 mm
- net Net-(D1-A): track 0.00 -> 8.39 mm
- net VBUS: track 89.2 -> 81.1 mm

Commit message: feat(hw):Added_TPS2116DRL
Parts:
- removed C25, C9: 10uF, Capacitor_SMD:C_0603_1608Metric
- removed D1: MBR120, Diode_SMD:D_SOD-123F
- removed Q3: DMG3415U-7, Package_TO_SOT_SMD:SOT-23
- added C7: 10uF, Capacitor_SMD:C_0603_1608Metric, B.Cu at (128.8, 96.6)
- added C8: 10uF, Capacitor_SMD:C_0603_1608Metric, B.Cu at (122.4, 96.7)
- added R10: 4.7k, Resistor_SMD:R_0603_1608Metric, B.Cu at (125.3, 93.7)
- added R12: 10k, Resistor_SMD:R_0603_1608Metric, B.Cu at (128.2, 92.2)
- added U7: TPS2116DRL, Package_TO_SOT_SMD:SOT-583-8, B.Cu at (125.3, 91.6)
- R5: value 100K -> 10k
- moved R5 3.69 mm to (123.2, 90.1), turned to 90 degrees
Connections:
- R5 pad 1: Net-(D1-A) -> Net-(SW3A-A)
- R5 pad 2: GND -> Net-(U7-ST)
- SW3 pad 1: Net-(D1-K) -> Net-(SW3A-A)
- U2 pad 5: Net-(D1-A) -> /Vref
Routing:
- net Net-(SW3A-A): track 0.00 -> 12.4 mm
- net Net-(D1-K): track 12.0 -> 0.00 mm
- net Net-(D1-A): track 8.39 -> 0.00 mm
- net /Vref: track 0.00 -> 7.91 mm
- net +3.3V: track 40.7 -> 47.6 mm, vias 0 -> 5
- net /PR1: track 0.00 -> 2.77 mm
- net Net-(U7-ST): track 0.00 -> 2.76 mm
- net GND: track 18.1 -> 20.2 mm, vias 85 -> 86
- net VBUS: track 81.1 -> 82.9 mm, vias 6 -> 8
- added copper zone on B.Cu, net +3.3V
- added copper zone on F.Cu, net +3.3V

Commit message: feat(Hw):Update_Schematic_And_Route
Parts:
- added C9: 100nF, Capacitor_SMD:C_0603_1608Metric, B.Cu at (121.8, 90.1)
