File: hardware/Badge-Pwnterrey-2026.kicad_pcb (KiCad board)
At the start: 2 copper layers, 75.5 x 60.2 mm, 65 parts, among them J1 Conn_01x08_Socket, J2 Conn_01x08_Socket, J3 Conn_01x10_Socket, J5 Conn_01x10_Socket, P1 USB_C_Plug_USB2.0, Q1 DMP2004TK-7, Q2 DMP2004TK-7, SW1 RESET, SW2 GPIO, SW3 On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

Commit message: feat(Hw):GPS_Pins_Added
Parts:
- added J4: GPS, Connector_PinHeader_2.54mm:PinHeader_1x04_P2.54mm_Vertical, B.Cu at (178.0, 53.0)
Routing:
- net /GPS_TX: track 40.0 -> 73.0 mm
- net /GPS_RX: track 45.7 -> 62.1 mm
- net /LPUART_RX: track 63.8 -> 64.3 mm
- net GND: vias 86 -> 90
